File: small-fry-pcb.kicad_pcb (KiCad board)
At the start: 2 copper layers, 302 x 144.1 mm, 140 parts, among them U1 Pico

Commit message: fixed cols
Parts:
- moved U1 9.36 mm to (205.8, 46.2), turned to -45 degrees
Connections:
- U1 pad 10: col11 -> row3
- U1 pad 11: unconnected-(U1-GPIO8-Pad11)_1 -> row4
- U1 pad 22: row4 -> col14
- U1 pad 24: row3 -> col13
- U1 pad 25: row2 -> col12
- U1 pad 26: row1 -> col11
- U1 pad 27: row0 -> col10
- U1 pad 29: col7 -> col9
- U1 pad 32: col9 -> col7
- U1 pad 34: col10 -> unconnected-(U1-GPIO28_ADC2-Pad34)_1
- U1 pad 6: col14 -> row0
- U1 pad 7: col13 -> row1
- U1 pad 9: col12 -> row2
Routing:
- net col8: track 118.5 -> 151.5 mm
- net col7: track 80.9 -> 110.6 mm
- net col9: track 134.8 -> 159.0 mm
- net row0: track 307.3 -> 289.2 mm
- net row1: track 324.6 -> 308.5 mm
- net col5: track 138.2 -> 122.9 mm
- net col10: track 157.4 -> 171.9 mm
- net col3: track 165.6 -> 151.7 mm
- net row2: track 303.6 -> 289.8 mm
- net col4: track 130.0 -> 116.5 mm
- net col11: track 182.5 -> 194.2 mm, vias 1 -> 0
- net row3: track 320.8 -> 309.3 mm
- net col0: track 216.0 -> 208.6 mm
- net row4: track 377.2 -> 370.1 mm
- net col12: track 202.6 -> 209.6 mm, vias 1 -> 0
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Other:
- board outline removed
