File: small-fry-pcb.kicad_pcb (KiCad board)
At the start: 2 copper layers, 338.4 x 100.6 mm, 143 parts, among them U1 Pico

Commit message: updated footprints, rotated mcu
Parts:
- moved G*** 279.3 mm to (62.6, 17.4) (x2)
- moved U1 181.5 mm to (208.9, 10.1), turned to -60 degrees
Routing:
- net col14: track 497.9 -> 0.00 mm
- net col13: track 477.0 -> 0.00 mm
- net col12: track 451.5 -> 0.00 mm
- net col11: track 428.6 -> 0.00 mm
- net col10: track 396.3 -> 0.00 mm
- net col9: track 373.6 -> 0.00 mm
- net row4: track 347.1 -> 0.00 mm
- net col8: track 339.6 -> 0.00 mm
- net row0: track 325.9 -> 0.00 mm
- net col7: track 321.4 -> 0.00 mm
- net row1: track 309.2 -> 0.00 mm
- net col6: track 298.7 -> 0.00 mm
- net row2: track 295.5 -> 0.00 mm
- net row3: track 292.3 -> 0.00 mm
- net col5: track 273.2 -> 0.00 mm
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Other:
- board outline removed
- board text removed: "GP15"

Commit message: Squashed commit of the following:
commit e493926800ae8eeeb9c8551a418d401659cc4f4a
Author: anchovie-codes <littlebrother.free@gmail.com>
Date:   Sun Nov 10 19:39:24 2024 -0500

    updated edge cuts and gerbers

commit a852bf54e9e750d94bc40db8a16316f7cdac5ac1
Author: anchovie-codes <littlebrother.free@gmail.com>
Date:   Sat Sep 28 17:49:30 2024 -0400

    fixed rows, generated gerbers

commit 9d77bf2fb49dd0b8cbfb8cfda25d822d23244967
Author: anchovie-codes <littlebrother.free@gmail.com>
Date:   Sat Sep 28 13:01:13 2024 -0400

    fixed cols

commit 5f5487953ddbebd1258b34876b9f208a7da505d8
Author: anchovie-codes <littlebrother.free@gmail.com>
Date:   Fri Sep 27 21:14:36 2024 -0400

    made it a fish
Parts:
- removed the G*** at (33.0, 92.5) (x2)
- removed the G*** at (62.6, 17.4)
- moved G*** 183.5 mm to (186.5, 152.8)
- moved D37 42.0 mm to (196.2, 118.9)
- moved D41 42.0 mm to (272.4, 118.9)
- moved D42 42.0 mm to (291.5, 118.9)
- moved D43 42.0 mm to (310.5, 118.9)
- moved D44 42.0 mm to (334.3, 118.9)
- moved D65 42.0 mm to (272.4, 157.0)
- moved MX37 42.0 mm to (188.2, 117.9)
- moved MX41 42.0 mm to (264.4, 117.9)
- moved MX42 42.0 mm to (283.5, 117.9)
- moved MX43 42.0 mm to (302.5, 117.9)
- moved MX44 42.0 mm to (326.3, 117.9)
- moved MX65 42.0 mm to (264.4, 156.0)
- moved D11 42.0 mm to (272.4, 80.8)
- moved D12 42.0 mm to (291.5, 80.8)
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Connections:
- U1 pad 1: col14 -> unconnected-(U1-GPIO0-Pad1)
- U1 pad 10: col7 -> row3
- U1 pad 11: col6 -> row4
- U1 pad 12: col5 -> col6
- U1 pad 14: col4 -> col5
- U1 pad 15: col3 -> col4
- U1 pad 16: col2 -> col3
- U1 pad 17: col1 -> col2
- U1 pad 19: col0 -> col1
- U1 pad 2: col13 -> unconnected-(U1-GPIO1-Pad2)_1
- U1 pad 20: unconnected-(U1-GPIO15-Pad20) -> col0
- U1 pad 22: row4 -> col14
- U1 pad 24: row3 -> col13
- U1 pad 25: row2 -> col12
- U1 pad 26: row1 -> col11
- U1 pad 27: row0 -> col10
- U1 pad 29: unconnected-(U1-GPIO22-Pad29) -> col9
- U1 pad 31: unconnected-(U1-GPIO26_ADC0-Pad31) -> col8
- U1 pad 32: unconnected-(U1-GPIO27_ADC1-Pad32) -> col7
- U1 pad 4: col12 -> unconnected-(U1-GPIO2-Pad4)_1
- U1 pad 5: col11 -> unconnected-(U1-GPIO3-Pad5)
- U1 pad 6: col10 -> row0
- U1 pad 7: col9 -> row1
- U1 pad 9: col8 -> row2
Routing:
- net row4: track 0.00 -> 412.3 mm, vias 0 -> 2
- net row1: track 0.00 -> 361.3 mm, vias 0 -> 2
- net row2: track 0.00 -> 356.4 mm, vias 0 -> 2
- net row3: track 0.00 -> 354.2 mm, vias 0 -> 2
- net row0: track 0.00 -> 344.6 mm
- net col14: track 0.00 -> 245.9 mm
- net col13: track 0.00 -> 225.3 mm
- net col0: track 0.00 -> 209.8 mm
- net col12: track 0.00 -> 209.6 mm
- net col11: track 0.00 -> 194.2 mm
- net col1: track 0.00 -> 186.4 mm
- net col10: track 0.00 -> 171.9 mm
- net col2: track 0.00 -> 168.2 mm
- net col9: track 0.00 -> 159.0 mm
- net col3: track 0.00 -> 151.9 mm
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Other:
- board outline added: 302.4 x 150.5 mm
